File: psu/lab_ps_with_atx_psu/lab_ps_with_atx_psu.sch (KiCad schematic (older format))
At the start: 32 parts, among them CON1 +5V StandBy, CON2 +5V DC PSU IN, J1 ExtPWR_LED, J2 RJ12_FTDI, J3 SPI Header, J4 i2C_BUS, SW1 RESET, U1 MCP1702-T3302E/CB, U2 ATmega328P-PU, U3 ADR5040, Y1 16MHz

Commit message: working on psu piece
Parts:
- added C10, C11, C12: 100n, Capacitor_SMD:C_0805_2012Metric_Pad1.15x1.40mm_HandSolder, symbol lab_ps_with_atx_psu-rescue:C_Small-Device
- added C13: 10u, Capacitor_SMD:CP_Elec_5x5.3, symbol lab_ps_with_atx_psu-rescue:CP_Small-Device
- added D5: SK33A, symbol Device:D_Schottky
- added R10, R11, R12, R13, R14, R15, R16, R17, R18, R19, R20, R9: 10, Resistor_THT:R_Axial_DIN0207_L6.3mm_D2.5mm_P7.62mm_Horizontal, symbol Device:R_Small
- added R21, R22, R23, R24: 18.2k, Resistor_THT:R_Axial_DIN0207_L6.3mm_D2.5mm_P7.62mm_Horizontal, symbol Device:R_Small
- added U4: INA219, Package_TO_SOT_SMD:SOT-23-8_Handsoldering, symbol INA219:INA219
- added U5: LM358, Package_DIP:DIP-8_W7.62mm_Socket_LongPads, symbol Amplifier_Operational:LM358
- added U6: MCP4726, Package_TO_SOT_SMD:SOT-23-6_Handsoldering, symbol MCP4726:MCP4726
- added U7: LT3080xT, Package_TO_SOT_THT:TO-220-5_P3.4x3.7mm_StaggerOdd_Lead3.8mm_Vertical, symbol Regulator_Linear:LT3080xT
- C9: renamed from C8; value 220u/35V -> 220u
Connections:
- net +12V: now also R10.2, R11.2, R12.2, R13.2, R14.2, R15.2, R16.2, R17.2, R18.2, R19.2, R9.2
- net +5V: now also C10.1, C12.2, U4.4 (VCC), U5.8 (V+), U6.2 (GND), U7.4 (VCONTROL)
- net Earth: now also C10.2, C12.1, C13.2, R24.1, U4.3 (GND), U4.7 (A0), U4.8 (A1), U5.4 (V-), U6.3 (VCC)
- net SCL: now also U4.6 (SDA), U6.7 (SCL)
- net SDA: now also U4.5 (SCL), U6.5 (SDA)
- net VREF: now also U6.6 (VREF)
- net ISET_PWM: now reaches U2.15 (PB1)
- new net: C11.1, R19.1, R23.2, U4.1 (VIN+)
- new net: C11.2, R20.1, U4.2 (VIN-)
- new net: C13.1, D5.1 (K), R10.1, R11.1, R12.1, R13.1, R14.1, R15.1, R16.1, R17.1, R18.1, R20.2, R9.1, U5.3 (+), U7.5 (IN)
- new net: R21.2, U5.1, U5.2 (-)
- new net: R23.1, R24.2, U5.5 (+)
- new net: R21.1, R22.2, U5.6 (-)
- new net: R22.1, U5.7
- no-connect marks 0 -> 1
Other:
- note added: "0-2.048V OUT"
- note added: "1R 6W shunt\n1mA = 1mV"
- note added: "Current Sense OUT\n1mV = 1mA"
- note added: "i2C Addr\n1000000"

Commit message: analog piece
Parts:
- added C13, C14, C15 (x2), C16: 100n, Capacitor_SMD:C_0805_2012Metric_Pad1.15x1.40mm_HandSolder, symbol lab_ps_with_atx_psu-rescue:C_Small-Device
- added Q1, Q2: 2N3904, Package_TO_SOT_THT:TO-92_Inline, symbol Transistor_BJT:2N3904
- added R26, R27: 18.2k, Resistor_THT:R_Axial_DIN0207_L6.3mm_D2.5mm_P7.62mm_Horizontal, symbol Device:R_Small
- added R28: 1k, Resistor_THT:R_Axial_DIN0207_L6.3mm_D2.5mm_P7.62mm_Horizontal, symbol Device:R_Small
- added R29, R35, R36: 1k, Resistor_SMD:R_0805_2012Metric_Pad1.15x1.40mm_HandSolder, symbol lab_ps_with_atx_psu-rescue:R-Device
- added R30, R31, R33, R34: 10k, Resistor_SMD:R_0805_2012Metric_Pad1.15x1.40mm_HandSolder, symbol lab_ps_with_atx_psu-rescue:R-Device
- added R32: 4k7, Resistor_SMD:R_0805_2012Metric_Pad1.15x1.40mm_HandSolder, symbol lab_ps_with_atx_psu-rescue:R-Device
- added unit 2 of U7
- added unit 3 of U7
- D5: value SK33A -> SK315SMA; footprint (none) -> Diode_SMD:D_SMA_Handsoldering; PN (none) -> 1003.7765; Price (none) -> 33; Supplier (none) -> hestore
Connections:
- net +5V: now also U6.3 (VCC), C13.1, C14.2, U7.8 (V+); no longer U6.2 (GND)
- net Earth: now also U6.2 (GND), C13.2, C14.1, C15.2, C15.2, C16.2, Q1.1 (E), Q2.1 (E), R28.2, R32.2, U7.4 (V-); no longer U6.3 (VCC)
- net ISET_PWM: now also R31.1
- net CLIM: now reaches U2.13 (PD7)
- net CLIM: now also Q1.3 (C)
- net at R22.1, U5.7: now also R29.1
- net at U6.1 (VOUT): now also U7.3 (+)
- net at U7.2 (SET): now also Q2.3 (C), R35.2, R36.2
- net at U7.3 (OUT): now also D5.2 (A)
- new net: C15.1, R29.2, U7.5 (+)
- new net: C15.1, R30.2, U7.6 (-)
- new net: R33.1, R34.1, U7.7
- new net: R35.1, U7.1
- new net: R26.2, R27.2, R28.1, U7.2 (-)
- new net: R26.1, R27.1, R36.1
- new net: C16.1, R30.1, R31.2, R32.1
- new net: Q1.2 (B), R33.2
- new net: Q2.2 (B), R34.2
