File: mysensors/ms-laki-thb-2chswitch/ms-laki-thb-2chswitch.sch (KiCad schematic (older format))
At the start: 3 parts, among them J1 230VAC_IN

Commit message: .
Parts:
- added C1: 100u, Capacitor_THT:CP_Radial_D8.0mm_P3.50mm, symbol Device:CP_Small
- added C10, C4: 10u, Capacitor_THT:CP_Radial_D4.0mm_P1.50mm, symbol Device:CP_Small
- added C11, C12, C13, C2, C3, C5, C8, C9: 100n, Capacitor_SMD:C_0805_2012Metric_Pad1.15x1.40mm_HandSolder, symbol Device:C_Small
- added C6, C7: 22p, Capacitor_THT:C_Disc_D3.0mm_W1.6mm_P2.50mm, symbol Device:C_Small
- added D1: 5VPWR, Diode_SMD:D_0805_2012Metric_Pad1.15x1.40mm_HandSolder, symbol Device:LED_Small
- added D2: 3_3VPWR, Diode_SMD:D_0805_2012Metric_Pad1.15x1.40mm_HandSolder, symbol Device:LED_Small
- added D3: SCK, Diode_SMD:D_0805_2012Metric_Pad1.15x1.40mm_HandSolder, symbol Device:LED_Small
- added D4: RELAY1, Diode_SMD:D_0805_2012Metric_Pad1.15x1.40mm_HandSolder, symbol Device:LED_Small
- added D5: 1N4148WS, Diode_SMD:D_SOD-323_HandSoldering, symbol Device:D_Small
- added J2: ICSP, Connector_PinHeader_2.54mm:PinHeader_2x03_P2.54mm_Vertical, symbol Connector_Generic:Conn_02x03_Odd_Even
- added J3: FTDI, Connector_PinSocket_2.54mm:PinSocket_1x06_P2.54mm_Vertical, symbol Connector:Conn_01x06_Male
- added J4: toBME280, symbol Connector:Conn_01x04_Male
- added K?: G5LE-1, Relay_THT:Relay_SPDT_Omron-G5LE-1, symbol Relay:G5LE-1
- added PS11: HLK-PM01, Converter_ACDC:Converter_ACDC_HiLink_HLK-PMxx, symbol Converter_ACDC:HLK-PM01
- added Q1: BC547B, Package_TO_SOT_THT:TO-92_HandSolder, symbol Transistor_BJT:BC547
- added R1, R4, R7: 1k, Resistor_SMD:R_0805_2012Metric_Pad1.15x1.40mm_HandSolder, symbol Device:R_Small
- added R2: 330, Resistor_SMD:R_0805_2012Metric_Pad1.15x1.40mm_HandSolder, symbol Device:R_Small
- added R3, R5, R6: 10k, Resistor_SMD:R_0805_2012Metric_Pad1.15x1.40mm_HandSolder, symbol Device:R_Small
- added R8: 510, Resistor_SMD:R_0805_2012Metric_Pad1.15x1.40mm_HandSolder, symbol Device:R_Small
- added RV1: 17VAC 250A/20usec, Varistor:RV_Disc_D7mm_W3.4mm_P5mm, symbol Device:Varistor
- added SW1: RESET, Button_Switch_SMD:SW_SPST_CK_RS282G05A3, symbol Switch:SW_Push
- added U1: MCP1702 T-3302E, Package_TO_SOT_SMD:SOT-23_Handsoldering, symbol Regulator_Linear:MCP1700-3302E_SOT23
- added U2: ATmega328P-PU, Package_DIP:DIP-28_W7.62mm_Socket, symbol MCU_Microchip_ATmega:ATmega328P-PU
- added U3: NRF24L01, RF_Module:nRF24L01_Breakout, symbol RF:NRF24L01_Breakout
- added U4: PC817, Package_DIP:DIP-4_W7.62mm, symbol Isolator:PC817
- added Y1: 16MHz, Crystal:Crystal_HC49-U_Vertical, symbol Device:Crystal_Small
- F2: value 2A Fast -> Termal 73C 10A; footprint (none) -> Fuse:Fuse_Bourns_MF-RG300; PN (none) -> 1002.3778; Price[HUF] (none) -> 115; Supplier (none) -> hestore
- J1: footprint (none) -> Connector_Wago:Wago_734-133_1x03_P3.50mm_Vertical; PN (none) -> 1002.6645; Price[HUF] (none) -> 108; Supplier (none) -> hestore
Connections:
- net at J1.1 (Pin_1): now also PS11.2 (AC/N), RV1.2
- net at J1.3 (Pin_3): now also F1.1
- net at F1.2: now also F2.1
- net at F2.2: now also PS11.1 (AC/L), RV1.1
- new net: D1.1 (K), R1.1
- new net: D2.1 (K), R2.1
- new net: C7.1, U2.10 (XTAL2/PB7), Y1.2
- new net: C5.1, U2.21 (AREF)
- new net: C6.1, U2.9 (XTAL1/PB6), Y1.1
- new net: D3.1 (K), R4.1
- new net: C11.2, J3.6 (Pin_6)
- new net: D4.1 (K), U4.1
- new net: R7.1, U4.2
- new net: R8.2, U4.3
- new net: Q1.2 (B), R8.1
- new net: D5.2 (A), Q1.1 (C)
- new net +3V3: C10.1, C3.1, C4.1, D2.2 (A), U1.2 (VO), U3.2 (VCC)
- new net +5V: C1.1, C12.2, C13.1, C2.1, C9.2, D1.2 (A), D5.1 (K), J2.2 (Pin_2), J3.3 (Pin_3), J4.1 (Pin_1), PS11.4 (+Vout), R3.1, R5.1, R6.1, U1.3 (VI), U2.20 (AVCC), U2.7 (VCC), U4.4
- new net CE: U2.15 (PB1), U3.3 (CE)
- new net CSN: U2.16 (PB2), U3.4 (~CSN)
- new net GNDA: C1.2, C10.2, C12.1, C13.2, C2.2, C3.2, C4.2, C5.2, C6.2, C7.2, C8.2, C9.1, J2.6 (Pin_6), J3.1 (Pin_1), J3.2 (Pin_2), J4.2 (Pin_2), PS11.3 (-Vout), Q1.3 (E), R1.2, R2.2, R4.2, R7.2, SW1.2, U1.1 (GND), U2.22 (GND), U2.8 (GND), U3.1 (GND)
- new net IRQ: U2.4 (PD2), U3.8 (IRQ)
- new net MISO: J2.1 (Pin_1), U2.18 (PB4), U3.7 (MISO)
- new net MOSI: J2.4 (Pin_4), U2.17 (PB3), U3.6 (MOSI)
- new net RELAY1: D4.2 (A), U2.6 (PD4)
- new net RELAY2: U2.11 (PD5)
- new net RESET: C11.1, C8.1, J2.5 (Pin_5), R3.2, SW1.1, U2.1 (~RESET~/PC6)
- new net RXD: J3.4 (Pin_4), U2.2 (PD0)
- new net SCK: D3.2 (A), J2.3 (Pin_3), U2.19 (PB5), U3.5 (SCK)
- new net SCL: J4.3 (Pin_3), R5.2, U2.28 (PC5)
- new net SDA: J4.4 (Pin_4), R6.2, U2.27 (PC4)
- new net TXD: J3.5 (Pin_5), U2.3 (PD1)
Other:
- moved on the sheet: F2

Commit message: .
Parts:
- removed K?: G5LE-1, Relay_THT:Relay_SPDT_Omron-G5LE-1, symbol Relay:G5LE-1
- added D6: RELAY1, Diode_SMD:D_0805_2012Metric_Pad1.15x1.40mm_HandSolder, symbol Device:LED_Small
- added D7: 1N4148WS, Diode_SMD:D_SOD-323_HandSoldering, symbol Device:D_Small
- added F3, F4: 5A Slow, Fuse:Fuseholder_Cylinder-5x20mm_Stelvio-Kontek_PTF78_Horizontal_Open, symbol Device:Fuse_Small
- added J5: Circ1, TerminalBlock_4Ucon:TerminalBlock_4Ucon_1x02_P3.50mm_Vertical, symbol Connector:Screw_Terminal_01x02
- added J6: Circ2, TerminalBlock_4Ucon:TerminalBlock_4Ucon_1x02_P3.50mm_Vertical, symbol Connector:Screw_Terminal_01x02
- added K1, K2: SONGLE_SRD-05VDC-SL-C, Relay_THT:Relay_SPDT_SANYOU_SRD_Series_Form_C, symbol Relay_Songle:SONGLE_SRD-05VDC-SL-C
- added Q2: BC547B, Package_TO_SOT_THT:TO-92_HandSolder, symbol Transistor_BJT:BC547
- added R10: 510, Resistor_SMD:R_0805_2012Metric_Pad1.15x1.40mm_HandSolder, symbol Device:R_Small
- added R9: 1k, Resistor_SMD:R_0805_2012Metric_Pad1.15x1.40mm_HandSolder, symbol Device:R_Small
- added U5: PC817, Package_DIP:DIP-4_W7.62mm, symbol Isolator:PC817
- J1: footprint Connector_Wago:Wago_734-133_1x03_P3.50mm_Vertical -> TerminalBlock_4Ucon:TerminalBlock_4Ucon_1x03_P3.50mm_Vertical
- J2: Price[HUF] 0 -> (none)
- J4: footprint (none) -> Connector_PinSocket_2.54mm:PinSocket_1x04_P2.54mm_Vertical
- U4: PN (none) -> 1002.6029; Price[HUF] (none) -> 25; Supplier (none) -> hestore
Connections:
- net +5V: now also D7.1 (K), K1.5, K2.5, U5.4
- net GNDA: now also Q2.3 (E), R9.2
- net RELAY2: now also D6.2 (A)
- net at D5.2 (A), Q1.1 (C): now also K1.2
- new net: F3.1, K1.1
- new net: J5.1 (Pin_1), K1.4
- new net: F3.2, J5.2 (Pin_2)
- new net: D6.1 (K), U5.1
- new net: R9.1, U5.2
- new net: R10.2, U5.3
- new net: Q2.2 (B), R10.1
- new net: D7.2 (A), K2.2, Q2.1 (C)
- new net: F4.1, K2.1
- new net: J6.1 (Pin_1), K2.4
- new net: F4.2, J6.2 (Pin_2)
- no-connect marks 0 -> 8

Commit message: .
Parts:
- C10, C4: footprint Capacitor_THT:CP_Radial_D4.0mm_P1.50mm -> Capacitor_Tantalum_SMD:CP_EIA-6032-28_Kemet-C_Pad2.25x2.35mm_HandSolder; PN 1000.0404 -> 1002.3050; Price[HUF] 6.5 -> 45.55
- C11, C12, C13, C2, C3, C5, C8, C9: footprint Capacitor_SMD:C_0805_2012Metric_Pad1.15x1.40mm_HandSolder -> Capacitor_SMD:C_1206_3216Metric_Pad1.42x1.75mm_HandSolder; PN 1000.1122 -> 1000.0289; Price[HUF] 4.72 -> 11
- C6, C7: footprint Capacitor_THT:C_Disc_D3.0mm_W1.6mm_P2.50mm -> Capacitor_SMD:C_1206_3216Metric_Pad1.42x1.75mm_HandSolder; PN 1002.5995 -> 1000.0587; Price[HUF] 4 -> 6.3
- D1: footprint Diode_SMD:D_0805_2012Metric_Pad1.15x1.40mm_HandSolder -> Diode_SMD:D_1206_3216Metric_Pad1.42x1.75mm_HandSolder; PN 1003.4529 -> 1003.6588; Price[HUF] 12 -> 14.3
- D2: footprint Diode_SMD:D_0805_2012Metric_Pad1.15x1.40mm_HandSolder -> Diode_SMD:D_1206_3216Metric_Pad1.42x1.75mm_HandSolder; PN 1003.4529 -> 1003.6591; Price[HUF] 12 -> 14.3
- D3: footprint Diode_SMD:D_0805_2012Metric_Pad1.15x1.40mm_HandSolder -> Diode_SMD:D_1206_3216Metric_Pad1.42x1.75mm_HandSolder; PN 1003.2677 -> 1003.6591; Price[HUF] 11 -> 9.3
- D4, D6: footprint Diode_SMD:D_0805_2012Metric_Pad1.15x1.40mm_HandSolder -> Diode_SMD:D_1206_3216Metric_Pad1.42x1.75mm_HandSolder; PN 1002.5834 -> 1003.6590; Price[HUF] 13.18 -> 7.1
- D5, D7: footprint Diode_SMD:D_SOD-323_HandSoldering -> Diode_SMD:D_1206_3216Metric_Pad1.42x1.75mm_HandSolder; PN 1003.8803 -> 1002.9300; Price[HUF] 4.9 -> 11
- R1, R4, R7, R9: footprint Resistor_SMD:R_0805_2012Metric_Pad1.15x1.40mm_HandSolder -> Resistor_SMD:R_1206_3216Metric_Pad1.42x1.75mm_HandSolder; PN 1000.1157 -> 1000.0256; Price[HUF] 2.2 -> 2.3
- R10, R8: footprint Resistor_SMD:R_0805_2012Metric_Pad1.15x1.40mm_HandSolder -> Resistor_SMD:R_1206_3216Metric_Pad1.42x1.75mm_HandSolder; PN 1002.0174 -> 1003.5946; Price[HUF] 2.76 -> 3.52
- R2: footprint Resistor_SMD:R_0805_2012Metric_Pad1.15x1.40mm_HandSolder -> Resistor_SMD:R_1206_3216Metric_Pad1.42x1.75mm_HandSolder; PN 1000.1170 -> 1000.0487
- R3, R5, R6: footprint Resistor_SMD:R_0805_2012Metric_Pad1.15x1.40mm_HandSolder -> Resistor_SMD:R_1206_3216Metric_Pad1.42x1.75mm_HandSolder; PN 1000.1145 -> 1000.0297
