File: mysensors/ms-laki-thb-2chswitch/ms-laki-thb-2chswitch.kicad_pcb (KiCad board)
At the start: 2 copper layers, 53 parts, among them J1 230VAC_IN, J2 ICSP, J3 FTDI, J4 toBME280, J5 Circ1, J6 Circ2, K1 SONGLE_SRD-05VDC-SL-C, K2 SONGLE_SRD-05VDC-SL-C, Q1 BC547B, Q2 BC547B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

Commit message: .
Parts:
- C10, C4: footprint Capacitor_THT:CP_Radial_D4.0mm_P1.50mm -> Capacitor_Tantalum_SMD:CP_EIA-6032-28_Kemet-C_Pad2.25x2.35mm_HandSolder
- C11, C12, C13, C2, C3, C5, C8, C9: footprint Capacitor_SMD:C_0805_2012Metric_Pad1.15x1.40mm_HandSolder -> Capacitor_SMD:C_1206_3216Metric_Pad1.42x1.75mm_HandSolder
- C6, C7: footprint Capacitor_THT:C_Disc_D3.0mm_W1.6mm_P2.50mm -> Capacitor_SMD:C_1206_3216Metric_Pad1.42x1.75mm_HandSolder
- D1, D2, D3, D4, D6: footprint Diode_SMD:D_0805_2012Metric_Pad1.15x1.40mm_HandSolder -> Diode_SMD:D_1206_3216Metric_Pad1.42x1.75mm_HandSolder
- D5, D7: footprint Diode_SMD:D_SOD-323_HandSoldering -> Diode_SMD:D_1206_3216Metric_Pad1.42x1.75mm_HandSolder
- R1, R10, R2, R3, R4, R5, R6, R7, R8, R9: footprint Resistor_SMD:R_0805_2012Metric_Pad1.15x1.40mm_HandSolder -> Resistor_SMD:R_1206_3216Metric_Pad1.42x1.75mm_HandSolder
- moved C2 71.4 mm to (102.9, 16.5), turned to 90 degrees
- moved U1 70.7 mm to (108.0, 16.5), turned to 180 degrees
- moved R3 70.5 mm to (92.7, 11.4)
- moved Y1 68.7 mm to (86.4, 38.1), turned to 270 degrees
- moved C8 67.1 mm to (87.4, 14.0), turned to 180 degrees
- moved R1 65.1 mm to (77.5, 27.9)
- moved D5 60.9 mm to (62.2, 40.6), turned to 90 degrees
- moved D2 60.6 mm to (106.7, 25.4)
- moved D1 59.9 mm to (77.5, 31.8)
- moved D6 50.1 mm to (73.7, 76.2)
- moved C7 48.2 mm to (81.3, 41.9), turned to 90 degrees
- moved C6 47.5 mm to (81.3, 36.8), turned to 270 degrees
- moved R2 46.9 mm to (106.7, 29.2)
- moved SW1 45.0 mm to (95.2, 16.5)
- moved C4 43.4 mm to (108.0, 21.6), turned to 180 degrees
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