File: mysensors/ms-laki-thb-battery/ms-laki-thb-battery.kicad_pcb (KiCad board)
At the start: 2 copper layers, 36.8 x 62.2 mm, 27 parts, among them J1 BatteryIN, J2 toBME280, J3 FTDI, J4 ICSP, SW1 RESET, U1 MCP1640CH, U2 ATmega328-PU, U3 NRF24L01_Breakout, Y1 8Mhz

Commit message: .
Parts:
- moved C9 97.6 mm to (29.1, 51.4)
- moved C11 79.7 mm to (54.2, 59.6)
- moved C4 78.2 mm to (28.3, 64.3), turned to 90 degrees
- moved C7 76.6 mm to (49.8, 45.1), turned to 90 degrees
- moved C2 74.0 mm to (36.6, 28.1), turned to 270 degrees
- moved C3 71.7 mm to (28.3, 59.1), turned to 90 degrees
- moved C8 70.7 mm to (33.0, 33.1), turned to 180 degrees
- moved C12 70.1 mm to (29.2, 78.7), turned to 90 degrees
- moved R4 67.9 mm to (49.8, 40.0), turned to 90 degrees
- moved R3 67.2 mm to (33.0, 36.1)
- moved L1 65.0 mm to (55.0, 30.1), turned to 90 degrees
- moved C1 64.9 mm to (50.5, 32.0), turned to 90 degrees
- moved U1 64.0 mm to (49.7, 27.7), turned to 180 degrees
- moved R1 60.0 mm to (39.0, 27.2)
- moved C6 59.8 mm to (33.3, 52.2), turned to 90 degrees
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Routing:
- net Earth: track 0.00 -> 40.4 mm
- net Net-(C1-Pad1): track 0.00 -> 20.6 mm
- net +3V3: track 0.00 -> 13.1 mm
- net Net-(R1-Pad2): track 0.00 -> 5.23 mm
- net Net-(L1-Pad2): track 0.00 -> 4.72 mm
Other:
- net class Default: clearance 0.2 -> 0.15; trace_width 0.25 -> 0.1; via_dia 0.8 -> 0.6
- net class Power added: clearance 0.2, trace_width 0.25, via_dia 0.8, via_drill 0.4
- net class Small_Power added: clearance 0.15, trace_width 0.1, via_dia 0.6, via_drill 0.4
- rule trace_clearance: 0.2 -> 0.15
- rule trace_min: 0.2 -> 0.1
